File: Hardware/Basic/Top/pecoskiSmartWatch-BASIC-TOP.brd (EAGLE design)
At the start: 38 x 38 mm, 61 parts, among them SW3 SWITCH.MOM, SW4 SWITCH.MOM, U1 NRF52832_MODULE_MDBT42, U2 PCF8523, U3 FT231XS, Y1 32.768kHz, Y2 32.7680kHz

Commit message: Updated HW 2021_03_13 PM
Parts:
- removed C10, C4: 4.7u, LinnesLab-Passives:C0603
- removed C21, C6, C9: 1u, LinnesLab-Passives:C0603
- removed CHRG: MCP73831, LinnesLab-Power:SOT23-5
- removed LDO1: MIC5504, LinnesLab-Power:SOT23-5
- removed R3: 100k, LinnesLab-Passives:R0603
- removed R4: (no value), LinnesLab-Passives:R0603
- removed U2: PCF8523, LinnesLab-Clocks:SO8
- removed Y2: 32.7680kHz, LinnesLab-Clocks:2-SMD.NOLEAD.2.0MMTO1.2MM
- moved SW2 37.1 mm to (35.0, 15.1), turned to 180 degrees
- moved R10 37.0 mm to (35.5, 12.6), turned to 180 degrees
- moved C11 36.8 mm to (35.4, 9.00), turned to 0 degrees
- moved D3 36.3 mm to (35.1, 10.8), turned to 180 degrees
- moved SW1 32.1 mm to (35.0, 35.7)
- moved LED1 26.2 mm to (34.0, 20.5), turned to 270 degrees
- moved LED2 24.7 mm to (35.6, 20.5), turned to 270 degrees
- moved DEBUG1 23.7 mm to (35.2, 29.4), turned to 270 degrees
- moved R6 23.1 mm to (34.0, 23.7), turned to 90 degrees
- moved R7 21.2 mm to (35.7, 23.8), turned to 90 degrees
- moved C5 16.1 mm to (18.8, 22.6), turned to 90 degrees
- moved C3 15.6 mm to (17.2, 22.6), turned to 270 degrees
- moved Y1 11.4 mm to (20.5, 22.2), turned to 90 degrees
- moved R14 10.1 mm to (32.1, 19.0), flipped to the top, turned to 270 degrees
- moved C2 5.60 mm to (17.0, 29.1)
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Connections:
- removed net N$17: CHRG.5, R4.2
- removed net N$19: U2.2, Y2.P$1
- removed net N$20: U2.1, Y2.P$2
- removed net VBAT: U2.3
- net 3.3V: no longer C21.1, C9.1, LDO1.5, U2.8
- net D27/CHRG.STATUS: no longer CHRG.1, R3.1
- net GND: no longer C10.2, C21.2, C4.1, C6.1, C9.2, CHRG.2, LDO1.2, R4.1, U2.4
- net SCL: no longer U2.6
- net SDA: no longer U2.5
- net VIN: no longer C4.2, C6.2, CHRG.4, LDO1.1, LDO1.3, R3.2
- net VLIPO: no longer C10.1, CHRG.3
Routing:
- net RESET: track 0.00 -> 13.7 mm
- net SWO: track 0.00 -> 11.9 mm, vias 0 -> 1
- net VIN: track 16.0 -> 4.73 mm
- net SWCLK: track 0.00 -> 8.29 mm
- net LED2: track 0.00 -> 8.06 mm
- net N$2: track 0.00 -> 7.74 mm
- net N$6: track 0.00 -> 7.08 mm
- net N$4: track 1.99 -> 8.16 mm
- net N$17: track 5.28 -> 0.00 mm
- net LED1: track 0.00 -> 4.97 mm
- net GND: track 34.1 -> 38.7 mm, vias 15 -> 19
- net N$13: track 0.00 -> 4.12 mm
- net SWDIO: track 1.39 -> 5.11 mm
- net VLIPO: track 25.0 -> 21.8 mm
- net 3.3V: track 2.31 -> 0.00 mm, vias 1 -> 0
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