File: Hardware/Basic/Top/pecoskiSmartWatch-BASIC-TOP.sch (EAGLE design)
At the start: 29 parts, among them U2 NRF52832_MODULE_MDBT42

Commit message: Updated top board hardware Eagle
Parts:
- added C2, C5, C6: 1u, LinnesLab-Passives:CAPACITOR0603
- added C20, C21: 4.7u, LinnesLab-Passives:CAPACITOR0603
- added CHRG2: MCP73831, LinnesLab-Power:MCP73831
- added D4, D5: (no value), LinnesLab-DiscreteSemi:SCHOTTKY-USC
- added J2: (no value), LinnesLab-Connectors:CONN_02
- added LDO2: MIC5504, LinnesLab-Power:MIC5504
- added R11: (no value), LinnesLab-Passives:RESISTOR0603
- added R12, R13, R14, R15: 100k, LinnesLab-Passives:RESISTOR0603
- added R8, R9: 10k, LinnesLab-Passives:RESISTOR0603
- added SW1, SW2: SWITCH.MOM, LinnesLab-Switches:SWITCH.MOM
- added U4: PCF8523, LinnesLab-Clocks:PCF8523
- added USB2: USB.MICRO-BIGGERPADS, LinnesLab-Connectors:USB.MICRO-BIGGERPADS
- added XTAL3: 32.7680kHz, LinnesLab-Clocks:CRYSTALECS-.327-12.5-12-C-TR
Connections:
- new net BATT: R13.1, R14.2
- new net CHRG.STAT: CHRG2.STAT, R12.1
- new net N$17: CHRG2.PROG, R11.2
- new net N$19: U4.OSCO, XTAL3.1
- new net N$20: U4.OSCI, XTAL3.2
- new net SW1: SW1.1, SW2.1
- new net USB+: USB2.D+
- new net USB-: USB2.D-
- new net VIN: C21.2, C5.2, CHRG2.VIN, D4.C, D5.C, LDO2.EN, LDO2.IN, R12.2
- new net VLIPO: C20.1, CHRG2.VBAT, D4.A, J2.2, R13.2
- new net V_USB: D5.A, USB2.V+
- net 3.3V: now also C2.1, C6.1, LDO2.OUT, R15.2, R8.2, R9.2, U4.VDD
- net GND: now also C2.2, C20.2, C21.1, C5.1, C6.2, CHRG2.VSS, J2.1, LDO2.GND, R11.1, R14.1, R15.1, SW1.3, SW1.4, SW2.3, SW2.4, U4.VSS, USB2.GND, USB2.SHIELD
- net SCL: now also R8.1, U4.SCL
- net SDA: now also R9.1, U4.SDA
Other:
- note added: "Back-up battery if desired"
- note added: "Buttons"
- note added: "Cortext Debugger / Programmer"
- note added: "Digital Outputs CS.OLED RESET.OLED DC.OLED Digital Inputs 3x Buttons Charge Status Analog Inputs Battery Monitor Analog Outputs"
- note added: "I2C Address = 0x68h"
- note added: "Power Management"
- note added: "RTC"
- note added: "Real-Time Clock"
- note added: "SD Card"
- note added: "nRF52832 Module"
- moved on the sheet: C13, C14, C15, C16, C17, C18, C19, CORTEX1, D1, R5, R6, R7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

Commit message: Updated Eagle Hardware 2021_02_27
Parts:
- added C22: 100n, LinnesLab-Passives:CAPACITOR0603
- added C23, C24: 47p, LinnesLab-Passives:CAPACITOR0603
- added JP2: (no value), LinnesLab-Switches:JUMPER-SMT_2_NO_SILK
- added LED5: RED, LinnesLab-LED:LED0603
- added LED6: YELLOW, LinnesLab-LED:LED0603
- added R1, R2: 0, LinnesLab-Passives:RESISTOR0603
- added R17, R18: 27, LinnesLab-Passives:RESISTOR0603
- added R19, R20: 1k, LinnesLab-Passives:RESISTOR0603
- added U5: FT231XS, LinnesLab-DigitalIC:FT231XS
Connections:
- removed net BATT: R13.1, R14.2
- removed net CD1: SD2.CARD_DETECT
- removed net CHRG.STAT: CHRG2.STAT, R12.1
- removed net CS.OLED: U3./CS
- removed net DC.OLED: U3.DC/I2C_SA0
- removed net RESET.OLED: U3./RES
- removed net RXD: U2.P0.08
- removed net SD.CS: SD2.CS
- removed net SW1: SW1.1, SW2.1
- removed net TXD: U2.P0.06
- new net !CTS: JP2.2, U5.!CTS
- new net !DTR: U5.!DTR
- new net A4/BATT: R13.1, R14.2, U2.P0.28/AIN4
- new net A6/TIA: U2.P0.30/AIN6
- new net A7/PPG: U2.P0.31/AIN7
- new net D11/SW1: SW1.1, U2.P0.11
- new net D15/SW2: SW2.1, U2.P0.15
- new net D16/CS.OLED: U2.P0.16, U3./CS
- new net D27/CHRG.STATUS: CHRG2.STAT, R12.1, U2.P0.27
- new net D29/LED.CTRL: U2.P0.29/AIN5
- new net D3/RESET.OLED: U2.P0.03/AIN1, U3./RES
- new net D4/DC.OLED: U2.P0.04/AIN2, U3.DC/I2C_SA0
- new net D5/CD1: SD2.CARD_DETECT, U2.P0.05/AIN3
- new net D7/SD.CS: SD2.CS, U2.P0.07
- new net FT3V3: U5.3V3OUT
- new net N$23: R17.2, U5.USBDM
- new net N$24: R18.2, U5.USBDP
- new net N$25: LED5.C, R19.2
- new net N$26: LED6.C, R20.2
- new net RXD.FT: R2.1, U5.RXD
- new net RXD.NRF: R1.2, U2.P0.08
- new net RXLED: R19.1, U5.CBUS1
- new net TXD.FT: R1.1, U5.TXD
- new net TXD.NRF: R2.2, U2.P0.06
- new net TXLED: R20.1, U5.CBUS2
- net 3.3V: now also C22.2, LED5.A, LED6.A, U5.!RESET, U5.VCCIO
- net GND: now also C22.1, C23.2, C24.1, JP2.1, U5.GND@16, U5.GND@6
- net SCL: now also R9.1; no longer R8.1
- net SDA: now also R8.1; no longer R9.1
- net USB+: now also C23.1, R18.1
- net USB-: now also C24.2, R17.1
- net V_USB: now also U5.VCC
Other:
- note added: "Digital Output"
- note added: "FTDI Serial-to-USB Converter"
- note added: "I don't remember if CTS needs to be grounded or left floating so here's a jumper to ground so it can be configued either way dynamically."
- note added: "Notes"
- note added: "TXD goes to RX on the other device RXD goes to TX on the other device"
- moved on the sheet: C10, C11, C12, C14, C7, C8, C9, CORTEX1, D1, L2, LED3, LED4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

Commit message: HW Updates 2021/03/06
Parts:
- removed C22: 100n, LinnesLab-Passives:CAPACITOR0603
- removed C23, C24: 47p, LinnesLab-Passives:CAPACITOR0603
- removed D4: (no value), LinnesLab-DiscreteSemi:SCHOTTKY-USC
- removed LED5: RED, LinnesLab-LED:LED0603
- removed LED6: YELLOW, LinnesLab-LED:LED0603
- removed R19: 1k, LinnesLab-Passives:RESISTOR0603
- removed U5: FT231XS, LinnesLab-DigitalIC:FT231XS
- removed XTAL3: 32.7680kHz, LinnesLab-Clocks:CRYSTALECS-.327-12.5-12-C-TR
- added C1: 1u, LinnesLab-Passives:CAPACITOR0603
- added C3: (no value), LinnesLab-Passives:CAPACITOR0603
- added C4: 4.7u, LinnesLab-Passives:CAPACITOR0603
- added D3: (no value), LinnesLab-DiscreteSemi:SCHOTTKY-USC
- added J1: (no value), LinnesLab-Connectors:CONN_02
- added LED1: RED, LinnesLab-LED:LED0603
- added LED2: BLUE, LinnesLab-LED:LED0603
- added R10: 10k, LinnesLab-Passives:RESISTOR0603
- added U1: NRF52832_MODULE_MDBT42, LinnesLab-Microcontrollers:NRF52832_MODULE_MDBT42
- added XTAL1: 32.768kHz, LinnesLab-Clocks:CRYSTALECS-.327-12.5-12-C-TR
- C10: value 300p -> 4.7u
- C11: value 300p -> 100n
- C12: value 10u -> 47p; device LinnesLab-Passives:CAPACITOR0805 -> LinnesLab-Passives:CAPACITOR0603
- C13: value 2.2uF -> 47p; device LinnesLab-Passives:CAPACITOR0402 -> LinnesLab-Passives:CAPACITOR0603
- C14: value 100n -> 10uF
- C15: value 2.2uF -> 100n; device LinnesLab-Passives:CAPACITOR0402 -> LinnesLab-Passives:CAPACITOR0603
- C16: value 10uF -> 2.2uF; device LinnesLab-Passives:CAPACITOR0603 -> LinnesLab-Passives:CAPACITOR0402
- C2: value 1u -> 10u; device LinnesLab-Passives:CAPACITOR0603 -> LinnesLab-Passives:CAPACITOR0805
- C20: value 4.7u -> 2.2uF; device LinnesLab-Passives:CAPACITOR0603 -> LinnesLab-Passives:CAPACITOR0402
- C21: value 4.7u -> 1u
- C5: value 1u -> (none)
- C7: value 1u -> 300p
- C8: value (none) -> 300p
- C9: value (none) -> 1u
- J2: device LinnesLab-Connectors:CONN_02 -> LinnesLab-Connectors:CONN_07-1.27MM
- LED4: value BLUE -> YELLOW
- R1, R2: value 0 -> 10k
- R11: value (none) -> 10k
- R12, R13: value 100k -> 27
- R14: value 100k -> 390k
- R15: value 100k -> 1k
- R17, R18: value 27 -> 0
- R3: value 1k -> 100k
- R4: value 1k -> (none)
- R5, R8, R9: value 10k -> 100k
- R6: value 10k -> 1k
- R7: value 390k -> 1k
- SW1, SW2: value SWITCH.MOM -> (none); device LinnesLab-Switches:SWITCH.MOM -> LinnesLab-Switches:SPST-PTS830GG140-COPY.1-3
- SW3, SW4: value (none) -> SWITCH.MOM; device LinnesLab-Switches:SPST-PTS830GG140-COPY.1-3 -> LinnesLab-Switches:SWITCH.MOM
- U2: value NRF52832_MODULE_MDBT42 -> PCF8523; device LinnesLab-Microcontrollers:NRF52832_MODULE_MDBT42 -> LinnesLab-Clocks:PCF8523; DIGIKEY (none) -> 568-5306-1-ND; I2C_ADDRESS (none) -> 0x68h; MFN (none) -> PCF8523T/1,118; MFN_MANUFACTURER (none) -> NXP USA Inc.
- U3: value (none) -> FT231XS; device LinnesLab-Displays:DISP_OLED_UG-2864HSWEG01-NO-WRAPAROUND -> LinnesLab-DigitalIC:FT231XS
- U4: value PCF8523 -> (none); device LinnesLab-Clocks:PCF8523 -> LinnesLab-Displays:DISP_OLED_UG-2864HSWEG01-NO-WRAPAROUND; DIGIKEY 568-5306-1-ND -> (none); I2C_ADDRESS 0x68h -> (none); MFN PCF8523T/1,118 -> (none); MFN_MANUFACTURER NXP USA Inc. -> (none)
- XTAL2: value 32.768kHz -> 32.7680kHz; FREQ (none) -> 32.7680KHZ
- renumbered CHRG2 to CHRG, CORTEX1 to DEBUG1, D5 to D2, JP2 to JP1, L2 to L1, LDO2 to LDO1, R20 to R16, SD2 to SD1, USB2 to USB1
Connections:
- net !CTS: now also U3.!CTS; no longer U5.!CTS
- net !DTR: now also U3.!DTR; no longer U5.!DTR
- net 3.3V: now also C15.2, C2.2, C20.2, C21.1, C9.1, D3.C, J2.4, LED3.A, LED4.A, R1.2, R10.2, R2.2, U1.VDD, U3.!RESET, U3.VCCIO, U4.VBAT; no longer C12.2, C17.2, C2.1, C22.2, C6.1, D1.C, LED5.A, LED6.A, R15.2, R8.2, R9.2, U3.VBAT, U3.VDD, U5.!RESET, U5.VCCIO
- net A4/BATT: now also R8.1, R9.2, U1.P0.28/AIN4; no longer R13.1, R14.2, U2.P0.28/AIN4
- net A6/TIA: now also J2.6, U1.P0.30/AIN6; no longer U2.P0.30/AIN6
- net A7/PPG: now also J2.7, U1.P0.31/AIN7; no longer U2.P0.31/AIN7
- net D11/SW1: now also SW3.1, U1.P0.11; no longer SW1.1, U2.P0.11
- net D15/SW2: now also SW4.1, U1.P0.15; no longer SW2.1, U2.P0.15
- net D16/CS.OLED: now also U1.P0.16, U4./CS; no longer U2.P0.16, U3./CS
- net D27/CHRG.STATUS: now also R3.1, U1.P0.27; no longer R12.1, U2.P0.27
- net D29/LED.CTRL: now also J2.5, U1.P0.29/AIN5; no longer U2.P0.29/AIN5
- net D3/RESET.OLED: now also U1.P0.03/AIN1, U4./RES; no longer U2.P0.03/AIN1, U3./RES
- net D4/DC.OLED: now also U1.P0.04/AIN2, U4.DC/I2C_SA0; no longer U2.P0.04/AIN2, U3.DC/I2C_SA0
- net D5/CD1: now also U1.P0.05/AIN3; no longer U2.P0.05/AIN3
- net D7/SD.CS: now also U1.P0.07; no longer U2.P0.07
- net DFU: now also SW1.B, U1.P0.20; no longer SW3.B, U2.P0.20
- net DTR: now also C11.1; no longer C14.1
- net FRST: now also U1.P0.22; no longer U2.P0.22
- net FT3V3: now also U3.3V3OUT; no longer U5.3V3OUT
- net GND: now also C1.2, C13.2, C14.1, C15.1, C2.1, C20.1, C21.2, C3.1, C4.1, C5.2, C6.1, C8.2, J1.1, J2.3, LED1.C, LED2.C, R14.2, R4.1, R5.1, R9.1, SW1.A, SW2.B, SW3.3, SW3.4, SW4.3, SW4.4, U1.GND@1, U1.GND@2, U1.GND@3, U1.GND@4, U2.VSS, U3.GND@16, U3.GND@6, U4.BS0, U4.BS2, U4.NC(GND)@1, U4.NC(GND)@2, U4.VLSS; no longer C11.2, C16.1, C18.1, C2.2, C20.2, C21.1, C22.1, C23.2, C24.1, C5.1, C6.2, C8.1, J2.1, LED3.C, LED4.C, R14.1, R15.1, R6.1, R7.2, SW1.3, SW1.4, SW2.3, SW2.4, SW3.A, SW4.B, U2.GND@1, U2.GND@2, U2.GND@3, U2.GND@4, U3.BS0, U3.BS2, U3.NC(GND)@1, U3.NC(GND)@2, U3.VLSS, U3.VSS, U5.GND@16, U5.GND@6
- net LED1: now also R6.2, U1.P0.17; no longer R3.2, U2.P0.17
- net LED2: now also R7.2, U1.P0.19; no longer R4.2, U2.P0.19
- net MISO: now also U1.P0.14; no longer U2.P0.14
- net MOSI: now also U1.P0.13, U4.D1/SPI_SDIN/I2C_SDA; no longer U2.P0.13, U3.D1/SPI_SDIN/I2C_SDA
- net N$1: now also R11.2, U4.BS1; no longer R6.2, U3.BS1
- net N$10: now also LED2.A, R7.1; no longer LED4.A, R4.1
- net N$11: now also U1.DCC; no longer U2.DCC
- net N$12: now also C1.1, U1.DEC4; no longer C7.1, U2.DEC4
- net N$13: now also C14.2, U4.VCC; no longer C16.2, U3.VCC
- net N$15: now also C17.2, U4.VCOMH; no longer C18.2, U3.VCOMH
- net N$17: now also R4.2; no longer R11.2
- net N$19: now also U2.OSCO, XTAL2.1; no longer U4.OSCO, XTAL3.1
- net N$2: now also R14.1, U4.IREF; no longer R7.1, U3.IREF
- net N$20: now also U2.OSCI, XTAL2.2; no longer U4.OSCI, XTAL3.2
- net N$23: now also R12.2, U3.USBDM; no longer R17.2, U5.USBDM
- net N$24: now also R13.2, U3.USBDP; no longer R18.2, U5.USBDP
- net N$25: now also LED3.C, R15.2; no longer LED5.C, R19.2
- net N$26: now also LED4.C; no longer LED6.C
- net N$3: now also C18.2, U4.C2P; no longer C13.2, U3.C2P
- net N$4: now also C3.2, U1.P0.00/XL1, XTAL1.1; no longer C8.2, U2.P0.00/XL1, XTAL2.1
- net N$5: now also C18.1, U4.C2N; no longer C13.1, U3.C2N
- net N$6: now also C5.1, U1.P0.01/XL2, XTAL1.2; no longer C9.1, U2.P0.01/XL2, XTAL2.2
- net N$7: now also C16.2, U4.C1P; no longer C15.2, U3.C1P
- net N$8: now also C16.1, U4.C1N; no longer C15.1, U3.C1N
- net N$9: now also LED1.A, R6.1; no longer LED3.A, R3.1
- net P0.09/NFC1: now also C7.1, U1.P0.09; no longer C11.1, U2.P0.09
- net P0.10/NFC2: now also C8.1, U1.P0.10; no longer C10.1, U2.P0.10
- net RESET: now also C11.2, D3.A, R10.1, SW2.A, U1.P0.21/RESET; no longer C14.2, D1.A, R5.1, SW4.A, U2.P0.21/RESET
- net RXD.FT: now also R18.1, U3.RXD; no longer R2.1, U5.RXD
- net RXD.NRF: now also R17.2, U1.P0.08; no longer R1.2, U2.P0.08
- net RXLED: now also R15.1, U3.CBUS1; no longer R19.1, U5.CBUS1
- net SCK: now also U1.P0.12, U4.D0/SPI_SCLK/I2C_SCK; no longer U2.P0.12, U3.D0/SPI_SCLK/I2C_SCK
- net SCL: now also J2.2, R2.1, U1.P0.26, U2.SCL; no longer R9.1, U2.P0.26, U4.SCL
- net SDA: now also J2.1, R1.1, U1.P0.25, U2.SDA; no longer R8.1, U2.P0.25, U4.SDA
- net SWCLK: now also U1.SWDCLK; no longer U2.SWDCLK
- net SWDIO: now also U1.SWDIO; no longer U2.SWDIO
- net SWO: now also U1.P0.18/SWO; no longer U2.P0.18/SWO
- net TXD.FT: now also R17.1, U3.TXD; no longer R1.1, U5.TXD
- net TXD.NRF: now also R18.2, U1.P0.06; no longer R2.2, U2.P0.06
- net TXLED: now also U3.CBUS2; no longer U5.CBUS2
- net USB+: now also C13.1, R13.1; no longer C23.1, R18.1
- net USB-: now also C12.2, R12.1; no longer C24.2, R17.1
- net VIN: now also C4.2, C6.2, D1.C, R3.2; no longer C21.2, C5.2, D4.C, R12.2
- net VLIPO: now also C10.1, D1.A, J1.2, R8.2; no longer C20.1, D4.A, J2.2, R13.2
- net V_USB: now also U3.VCC; no longer U5.VCC
Other:
- note added: "Connection to bottom board"
- moved on the sheet: C10, C11, C12, C13, C14, C15, C16, C17, C18, C2, C20, C21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

Commit message: HW Updates 2021/03/06 Pt 2
Parts:
- removed C7, C8: 300p, LinnesLab-Passives:CAPACITOR0603
- removed R5: 100k, LinnesLab-Passives:RESISTOR0603
- renumbered XTAL1 to Y1, XTAL2 to Y2
Connections:
- net 3.3V: no longer R5.2
- net GND: no longer C7.2, C8.2, R5.1
- net P0.09/NFC1: no longer C7.1
- net P0.10/NFC2: no longer C8.1
Changed lines of the file:
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@@
 <part name="GND15" library="LinnesLab-Symbols" deviceset="GND" device=""/>
 <part name="GND16" library="LinnesLab-Symbols" deviceset="GND" device=""/>
-<part name="GND17" library="LinnesLab-Symbols" deviceset="GND" device=""/>
-<part name="GND18" library="LinnesLab-Symbols" deviceset="GND" device=""/>
 <part name="GND19" library="LinnesLab-Symbols" deviceset="GND" device=""/>
 <part name="GND20" library="LinnesLab-Symbols" deviceset="GND" device=""/>
@@
 <part name="C3" library="LinnesLab-Passives" deviceset="CAPACITOR" device="0603" package3d_urn="urn:adsk.eagle:package:15661989/2"/>
 <part name="C5" library="LinnesLab-Passives" deviceset="CAPACITOR" device="0603" package3d_urn="urn:adsk.eagle:package:15661989/2"/>
-<part name="C8" library="LinnesLab-Passives" deviceset="CAPACITOR" device="0603" package3d_urn="urn:adsk.eagle:package:15661989/2" value="300p"/>
-<part name="C7" library="LinnesLab-Passives" deviceset="CAPACITOR" device="0603" package3d_urn="urn:adsk.eagle:package:15661989/2" value="300p"/>
 <part name="C2" library="LinnesLab-Passives" deviceset="CAPACITOR" device="0805" package3d_urn="urn:adsk.eagle:package:15662010/2" value="10u"/>
 <part name="L1" library="LinnesLab-Passives" deviceset="INDUCTOR" device="0603" override_package3d_urn="urn:adsk.eagle:package:18592195/2" override_package_urn="urn:adsk.eagle:footprint:18592196/1" value="10u"/>
@@
 <part name="R6" library="LinnesLab-Passives" deviceset="RESISTOR" device="0603" package3d_urn="urn:adsk.eagle:package:15661944/2" value="1k"/>
 <part name="R7" library="LinnesLab-Passives" deviceset="RESISTOR" device="0603" package3d_urn="urn:adsk.eagle:package:15661944/2" value="1k"/>
-<part name="XTAL1" library="LinnesLab-Clocks" deviceset="CRYSTAL" device="ECS-.327-12.5-12-C-TR" package3d_urn="urn:adsk.eagle:package:18579459/2" value="32.768kHz"/>
+<part name="Y1" library="LinnesLab-Clocks" deviceset="CRYSTAL" device="ECS-.327-12.5-12-C-TR" package3d_urn="urn:adsk.eagle:package:18579459/2" value="32.768kHz"/>
 <part name="R10" library="LinnesLab-Passives" deviceset="RESISTOR" device="0603" package3d_urn="urn:adsk.eagle:package:15661944/2" value="10k"/>
 <part name="C11" library="LinnesLab-Passives" deviceset="CAPACITOR" device="0603" package3d_urn="urn:adsk.eagle:package:15661989/2" value="100n"/>
@@
 <part name="SUPPLY16" library="LinnesLab-Symbols" deviceset="VLIPO" device=""/>
 <part name="GND43" library="LinnesLab-Symbols" deviceset="GND" device=""/>
-<part name="R5" library="LinnesLab-Passives" deviceset="RESISTOR" device="0603" package3d_urn="urn:adsk.eagle:package:15661944/2" value="100k"/>
-<part name="GND44" library="LinnesLab-Symbols" deviceset="GND" device=""/>
 <part name="SUPPLY17" library="LinnesLab-Symbols" deviceset="VIN" device=""/>
 <part name="GND3" library="LinnesLab-Symbols" deviceset="GND" device=""/>
@@
 <part name="C21" library="LinnesLab-Passives" deviceset="CAPACITOR" device="0603" package3d_urn="urn:adsk.eagle:package:15661989/2" value="1u"/>
 <part name="SUPPLY11" library="LinnesLab-Symbols" deviceset="3.3V" device=""/>
-<part name="XTAL2" library="LinnesLab-Clocks" deviceset="CRYSTAL" device="ECS-.327-12.5-12-C-TR" package3d_urn="urn:adsk.eagle:package:18579459/2" value="32.7680kHz">
+<part name="Y2" library="LinnesLab-Clocks" deviceset="CRYSTAL" device="ECS-.327-12.5-12-C-TR" package3d_urn="urn:adsk.eagle:package:18579459/2" value="32.7680kHz">
 <attribute name="FREQ" value="32.7680KHZ"/>
 </part>
@@
 <attribute name="VALUE" x="114.3" y="190.246" size="1.778" layer="96" align="top-center"/>
 </instance>
-<instance part="GND17" gate="G$1" x="116.84" y="160.02" smashed="yes">
-<attribute name="VALUE" x="116.84" y="159.766" size="1.778" layer="96" align="top-center"/>
-</instance>
-<instance part="GND18" gate="G$1" x="104.14" y="160.02" smashed="yes">
-<attribute name="VALUE" x="104.14" y="159.766" size="1.778" layer="96" align="top-center"/>
-</instance>
 <instance part="GND19" gate="G$1" x="93.98" y="160.02" smashed="yes">
 <attribute name="VALUE" x="93.98" y="159.766" size="1.778" layer="96" align="top-center"/>
@@
 <attribute name="VALUE" x="95.504" y="165.481" size="1.778" layer="96"/>
 </instance>
-<instance part="C8" gate="G$1" x="116.84" y="167.64" smashed="yes">
-<attribute name="NAME" x="118.364" y="170.561" size="1.778" layer="95"/>
-<attribute name="VALUE" x="118.364" y="165.481" size="1.778" layer="96"/>
-</instance>
-<instance part="C7" gate="G$1" x="104.14" y="167.64" smashed="yes">
-<attribute name="NAME" x="105.664" y="170.561" size="1.778" layer="95"/>
-<attribute name="VALUE" x="105.664" y="165.481" size="1.778" layer="96"/>
-</instance>
 <instance part="C2" gate="G$1" x="73.66" y="203.2" smashed="yes" rot="R180">
 <attribute name="NAME" x="72.136" y="200.279" size="1.778" layer="95" rot="R180"/>
@@
 <attribute name="VALUE" x="155.702" y="209.55" size="1.778" layer="96" rot="R90"/>
 </instance>
-<instance part="XTAL1" gate="G$1" x="86.36" y="175.26" smashed="yes">
+<instance part="Y1" gate="G$1" x="86.36" y="175.26" smashed="yes">
 <attribute name="NAME" x="86.36" y="177.292" size="1.778" layer="95" font="vector" align="bottom-center"/>
 <attribute name="VALUE" x="86.36" y="173.228" size="1.778" layer="96" font="vector" align="top-center"/>
@@
 <attribute name="VALUE" x="124.46" y="-71.374" size="1.778" layer="96" align="top-center"/>
 </instance>
-<instance part="R5" gate="G$1" x="137.16" y="-35.56" smashed="yes" rot="R90">
-<attribute name="NAME" x="135.6614" y="-39.37" size="1.778" layer="95" rot="R90"/>
-<attribute name="VALUE" x="140.462" y="-39.37" size="1.778" layer="96" rot="R90"/>
-</instance>
-<instance part="GND44" gate="G$1" x="137.16" y="-45.72" smashed="yes">
-<attribute name="VALUE" x="137.16" y="-45.974" size="1.778" layer="96" align="top-center"/>
-</instance>
 <instance part="SUPPLY17" gate="G$1" x="78.74" y="-25.4" smashed="yes">
 <attribute name="VALUE" x="78.74" y="-22.606" size="1.778" layer="96" align="bottom-center"/>
@@
 <attribute name="VALUE" x="381" y="-50.546" size="1.778" layer="96" align="bottom-center"/>
 </instance>
-<instance part="XTAL2" gate="G$1" x="320.04" y="-58.42" smashed="yes">
+<instance part="Y2" gate="G$1" x="320.04" y="-58.42" smashed="yes">
 <attribute name="NAME" x="320.04" y="-56.388" size="1.778" layer="95" font="vector" align="bottom-center"/>
 <attribute name="FREQ" x="320.04" y="-58.42" size="1.27" layer="96" display="off"/>
@@
 <junction x="78.74" y="175.26"/>
 <pinref part="C3" gate="G$1" pin="2"/>
-<pinref part="XTAL1" gate="G$1" pin="1"/>
+<pinref part="Y1" gate="G$1" pin="1"/>
 <wire x1="78.74" y1="175.26" x2="83.82" y2="175.26" width="0.1524" layer="91"/>
 <pinref part="U1" gate="G$1" pin="P0.00/XL1"/>
@@
 <junction x="93.98" y="175.26"/>
 <pinref part="C5" gate="G$1" pin="1"/>
-<pinref part="XTAL1" gate="G$1" pin="2"/>
+<pinref part="Y1" gate="G$1" pin="2"/>
 <wire x1="93.98" y1="175.26" x2="88.9" y2="175.26" width="0.1524" layer="91"/>
 <pinref part="U1" gate="G$1" pin="P0.01/XL2"/>
@@
 <pinref part="GND20" gate="G$1" pin="GND"/>
 <pinref part="C3" gate="G$1" pin="1"/>
-</segment>
-<segment>
-<pinref part="C7" gate="G$1" pin="2"/>
-<pinref part="GND18" gate="G$1" pin="GND"/>
-<wire x1="104.14" y1="162.56" x2="104.14" y2="165.1" width="0.1524" layer="91"/>
-</segment>
-<segment>
-<pinref part="C8" gate="G$1" pin="2"/>
-<pinref part="GND17" gate="G$1" pin="GND"/>
-<wire x1="116.84" y1="162.56" x2="116.84" y2="165.1" width="0.1524" layer="91"/>
 </segment>
 <segment>
@@
 </segment>
 <segment>
-<pinref part="R5" gate="G$1" pin="1"/>
-<pinref part="GND44" gate="G$1" pin="GND"/>
-<wire x1="137.16" y1="-43.18" x2="137.16" y2="-40.64" width="0.1524" layer="91"/>
-</segment>
-<segment>
 <wire x1="325.12" y1="-66.04" x2="322.58" y2="-66.04" width="0.1524" layer="91"/>
 <wire x1="322.58" y1="-68.58" x2="322.58" y2="-66.04" width="0.1524" layer="91"/>
@@
 <wire x1="127" y1="-25.4" x2="127" y2="-27.94" width="0.1524" layer="91"/>
 <junction x="127" y="-27.94"/>
-<wire x1="127" y1="-27.94" x2="137.16" y2="-27.94" width="0.1524" layer="91"/>
-<pinref part="R5" gate="G$1" pin="2"/>
-<wire x1="137.16" y1="-27.94" x2="137.16" y2="-30.48" width="0.1524" layer="91"/>
 </segment>
 <segment>
@@
 <segment>
 <wire x1="109.22" y1="195.58" x2="109.22" y2="175.26" width="0.1524" layer="91"/>
-<wire x1="104.14" y1="175.26" x2="109.22" y2="175.26" width="0.1524" layer="91"/>
-<wire x1="104.14" y1="175.26" x2="104.14" y2="172.72" width="0.1524" layer="91"/>
-<pinref part="C7" gate="G$1" pin="1"/>
 <pinref part="U1" gate="G$1" pin="P0.09"/>
 <label x="109.22" y="177.8" size="1.27" layer="95" rot="R180" xref="yes"/>
@@
 <segment>
 <wire x1="111.76" y1="195.58" x2="111.76" y2="175.26" width="0.1524" layer="91"/>
-<wire x1="111.76" y1="175.26" x2="116.84" y2="175.26" width="0.1524" layer="91"/>
-<wire x1="116.84" y1="175.26" x2="116.84" y2="172.72" width="0.1524" layer="91"/>
-<pinref part="C8" gate="G$1" pin="1"/>
 <pinref part="U1" gate="G$1" pin="P0.10"/>
 <label x="111.76" y="177.8" size="1.27" layer="95" xref="yes"/>
@@
 <wire x1="314.96" y1="-60.96" x2="314.96" y2="-58.42" width="0.1524" layer="91"/>
 <wire x1="314.96" y1="-58.42" x2="317.5" y2="-58.42" width="0.1524" layer="91"/>
-<pinref part="XTAL2" gate="G$1" pin="1"/>
+<pinref part="Y2" gate="G$1" pin="1"/>
 <pinref part="U2" gate="G$1" pin="OSCO"/>
 </segment>
@@
 <segment>
 <wire x1="322.58" y1="-58.42" x2="325.12" y2="-58.42" width="0.1524" layer="91"/>
-<pinref part="XTAL2" gate="G$1" pin="2"/>
+<pinref part="Y2" gate="G$1" pin="2"/>
 <pinref part="U2" gate="G$1" pin="OSCI"/>
 </segment>
