File: Hardware/Basic/Top/pecoskiSmartWatch-BASIC-TOP.sch (EAGLE design)
At the start: 62 parts, among them SW3 SWITCH.MOM, SW4 SWITCH.MOM, U1 NRF52832_MODULE_MDBT42, U2 PCF8523, U3 FT231XS, Y1 32.768kHz, Y2 32.7680kHz

Commit message: Updated HW 2021_03_13 AM
Parts:
- removed SD1: (no value), LinnesLab-Connectors:MICROSD
Connections:
- removed net CD2: SD1.CARD_DETECT1
- net 3.3V: no longer SD1.VDD
- net D5/CD1: no longer SD1.CARD_DETECT
- net D7/SD.CS: no longer SD1.CS
- net GND: no longer SD1.GND, SD1.GND1, SD1.VSS
- net MISO: no longer SD1.DATA_OUT
- net MOSI: no longer SD1.DATA_IN
- net SCK: no longer SD1.SCLK
Other:
- note removed: "Connect MISO, MOSI, and SCK to appropriate pins on microcontroller. Those are SPI pins and are generally prespecified. You have more flexibility with the SD.CS pin."
- note removed: "SD Card"
Changed lines of the file:
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@@
 <part name="R11" library="LinnesLab-Passives" deviceset="RESISTOR" device="0603" package3d_urn="urn:adsk.eagle:package:15661944/2" value="10k"/>
 <part name="R14" library="LinnesLab-Passives" deviceset="RESISTOR" device="0603" package3d_urn="urn:adsk.eagle:package:15661944/2" value="390k"/>
-<part name="SUPPLY7" library="LinnesLab-Symbols" deviceset="3.3V" device=""/>
-<part name="GND22" library="LinnesLab-Symbols" deviceset="GND" device=""/>
-<part name="SD1" library="LinnesLab-Connectors" deviceset="MICROSD" device="" package3d_urn="urn:adsk.eagle:package:17873109/2"/>
 <part name="CHRG" library="LinnesLab-Power" deviceset="MCP73831" device=""/>
 <part name="LDO1" library="LinnesLab-Power" deviceset="MIC5504" device=""/>
@@
 advanced users only</text>
 <text x="350.52" y="137.16" size="4.318" layer="90" font="vector" ratio="15">OLED</text>
-<text x="210.82" y="-78.74" size="1.778" layer="97">Connect MISO, MOSI, and SCK
-to appropriate pins on
-microcontroller. Those are SPI
-pins and are generally prespecified.
-You have more flexibility with the
-SD.CS pin.</text>
 <text x="355.6" y="-71.12" size="1.27" layer="97">I2C Address = 0x68h</text>
 <text x="312.42" y="-71.12" size="1.27" layer="97">Back-up
@@
 <text x="365.76" y="144.78" size="5.08" layer="97" font="vector" ratio="15">OLED</text>
 <text x="78.74" y="-15.24" size="5.08" layer="97" font="vector" ratio="15">Power Management</text>
-<text x="218.44" y="0" size="5.08" layer="97" font="vector" ratio="15">SD Card</text>
 <text x="332.74" y="-2.54" size="5.08" layer="97" font="vector" ratio="15">Buttons</text>
 <text x="312.42" y="-43.18" size="5.08" layer="97" font="vector" ratio="15">Real-Time Clock</text>
@@
 <attribute name="VALUE" x="341.63" y="66.802" size="1.778" layer="96" rot="R180"/>
 </instance>
-<instance part="SUPPLY7" gate="G$1" x="213.36" y="-10.16" smashed="yes">
-<attribute name="VALUE" x="213.36" y="-7.366" size="1.778" layer="96" align="bottom-center"/>
-</instance>
-<instance part="GND22" gate="G$1" x="213.36" y="-58.42" smashed="yes">
-<attribute name="VALUE" x="213.36" y="-58.674" size="1.778" layer="96" align="top-center"/>
-</instance>
-<instance part="SD1" gate="G$1" x="233.68" y="-33.02" smashed="yes">
-<attribute name="NAME" x="218.44" y="-11.43" size="1.778" layer="95"/>
-<attribute name="VALUE" x="236.22" y="-11.43" size="1.778" layer="96"/>
-</instance>
 <instance part="CHRG" gate="G$1" x="111.76" y="-63.5" smashed="yes">
 <attribute name="NAME" x="104.14" y="-57.912" size="1.778" layer="95"/>
@@
 </segment>
 <segment>
-<wire x1="215.9" y1="-45.72" x2="213.36" y2="-45.72" width="0.1524" layer="91"/>
-<pinref part="GND22" gate="G$1" pin="GND"/>
-<wire x1="213.36" y1="-45.72" x2="213.36" y2="-50.8" width="0.1524" layer="91"/>
-<wire x1="213.36" y1="-50.8" x2="213.36" y2="-53.34" width="0.1524" layer="91"/>
-<wire x1="213.36" y1="-53.34" x2="213.36" y2="-55.88" width="0.1524" layer="91"/>
-<wire x1="215.9" y1="-50.8" x2="213.36" y2="-50.8" width="0.1524" layer="91"/>
-<junction x="213.36" y="-50.8"/>
-<wire x1="215.9" y1="-53.34" x2="213.36" y2="-53.34" width="0.1524" layer="91"/>
-<junction x="213.36" y="-53.34"/>
-<pinref part="SD1" gate="G$1" pin="VSS"/>
-<pinref part="SD1" gate="G$1" pin="GND"/>
-<pinref part="SD1" gate="G$1" pin="GND1"/>
-</segment>
-<segment>
 <pinref part="C6" gate="G$1" pin="1"/>
 <pinref part="GND34" gate="G$1" pin="GND"/>
@@
 </segment>
 <segment>
-<pinref part="SUPPLY7" gate="G$1" pin="3.3V"/>
-<wire x1="213.36" y1="-10.16" x2="213.36" y2="-43.18" width="0.1524" layer="91"/>
-<wire x1="213.36" y1="-43.18" x2="215.9" y2="-43.18" width="0.1524" layer="91"/>
-<pinref part="SD1" gate="G$1" pin="VDD"/>
-</segment>
-<segment>
 <pinref part="LDO1" gate="G$1" pin="OUT"/>
 <wire x1="121.92" y1="-27.94" x2="127" y2="-27.94" width="0.1524" layer="91"/>
@@
 <label x="337.82" y="83.82" size="1.27" layer="95" rot="R180" xref="yes"/>
 </segment>
-<segment>
-<wire x1="210.82" y1="-30.48" x2="215.9" y2="-30.48" width="0.1524" layer="91"/>
-<label x="210.82" y="-30.48" size="1.27" layer="95" rot="R180" xref="yes"/>
-<pinref part="SD1" gate="G$1" pin="SCLK"/>
-</segment>
 </net>
 <net name="MOSI" class="0">
@@
 <label x="337.82" y="81.28" size="1.27" layer="95" rot="R180" xref="yes"/>
 </segment>
-<segment>
-<wire x1="210.82" y1="-27.94" x2="215.9" y2="-27.94" width="0.1524" layer="91"/>
-<label x="210.82" y="-27.94" size="1.27" layer="95" rot="R180" xref="yes"/>
-<pinref part="SD1" gate="G$1" pin="DATA_IN"/>
-</segment>
 </net>
 <net name="MISO" class="0">
@@
 <pinref part="U1" gate="G$1" pin="P0.14"/>
 <label x="124.46" y="215.9" size="1.27" layer="95" xref="yes"/>
-</segment>
-<segment>
-<wire x1="210.82" y1="-25.4" x2="215.9" y2="-25.4" width="0.1524" layer="91"/>
-<label x="210.82" y="-25.4" size="1.27" layer="95" rot="R180" xref="yes"/>
-<pinref part="SD1" gate="G$1" pin="DATA_OUT"/>
 </segment>
 </net>
@@
 <pinref part="U4" gate="G$1" pin="VCOMH"/>
 <wire x1="347.98" y1="60.96" x2="330.2" y2="60.96" width="0.1524" layer="91"/>
-</segment>
-</net>
-<net name="CD2" class="0">
-<segment>
-<wire x1="210.82" y1="-17.78" x2="215.9" y2="-17.78" width="0.1524" layer="91"/>
-<label x="210.82" y="-17.78" size="1.27" layer="95" rot="R180" xref="yes"/>
-<pinref part="SD1" gate="G$1" pin="CARD_DETECT1"/>
 </segment>
 </net>
@@
 <label x="104.14" y="193.04" size="1.27" layer="95" rot="R270" xref="yes"/>
 </segment>
-<segment>
-<wire x1="210.82" y1="-33.02" x2="215.9" y2="-33.02" width="0.1524" layer="91"/>
-<label x="210.82" y="-33.02" size="1.27" layer="95" rot="R180" xref="yes"/>
-<pinref part="SD1" gate="G$1" pin="CS"/>
-</segment>
 </net>
 <net name="D5/CD1" class="0">
@@
 <label x="99.06" y="193.04" size="1.27" layer="95" rot="R270" xref="yes"/>
 </segment>
-<segment>
-<wire x1="210.82" y1="-15.24" x2="215.9" y2="-15.24" width="0.1524" layer="91"/>
-<label x="210.82" y="-15.24" size="1.27" layer="95" rot="R180" xref="yes"/>
-<pinref part="SD1" gate="G$1" pin="CARD_DETECT"/>
-</segment>
-</net>
+</net>

Commit message: Updated HW 2021_03_13 PM
Parts:
- removed C10, C4: 4.7u, LinnesLab-Passives:CAPACITOR0603
- removed C21, C6, C9: 1u, LinnesLab-Passives:CAPACITOR0603
- removed CHRG: MCP73831, LinnesLab-Power:MCP73831
- removed LDO1: MIC5504, LinnesLab-Power:MIC5504
- removed R3: 100k, LinnesLab-Passives:RESISTOR0603
- removed R4: (no value), LinnesLab-Passives:RESISTOR0603
- removed U2: PCF8523, LinnesLab-Clocks:PCF8523
- removed Y2: 32.7680kHz, LinnesLab-Clocks:CRYSTALECS-.327-12.5-12-C-TR
Connections:
- removed net N$17: CHRG.PROG, R4.2
- removed net N$19: U2.OSCO, Y2.1
- removed net N$20: U2.OSCI, Y2.2
- net 3.3V: no longer C21.1, C9.1, LDO1.OUT, U2.VDD
- net D27/CHRG.STATUS: no longer CHRG.STAT, R3.1
- net GND: no longer C10.2, C21.2, C4.1, C6.1, C9.2, CHRG.VSS, LDO1.GND, R4.1, U2.VSS
- net SCL: no longer U2.SCL
- net SDA: no longer U2.SDA
- net VIN: no longer C4.2, C6.2, CHRG.VIN, LDO1.EN, LDO1.IN, R3.2
- net VLIPO: no longer C10.1, CHRG.VBAT
Other:
- note removed: "Back-up battery if desired"
- note removed: "Digital Output"
- note removed: "I2C Address = 0x68h"
- note removed: "Real-Time Clock"
